File: PCB/Machine-Controller.kicad_pcb (KiCad board)
At the start: 4 copper layers, 43.1 x 37.7 mm, 85 parts, among them J1 RESET, J2 Conn_01x05, J3 Conn_01x03, J4 Conn_01x02, J5 Conn_01x03, J6 USB_C_Receptacle_USB2.0, J7 OUTPUT, Q1 SSM3J340R, SW1 SW_SPDT, SW2 SW_Push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

Commit message: BoM and Docs
Parts:
- removed FBr1: FerriteBead, Capacitor_SMD:C_0805_2012Metric
- removed J1: RESET, Personalised:SW_SPST_TL3342
- added SW4: BTN_R, Finn-Lib:SW_SPST_TL3342, F.Cu at (143.5, 97.3)
- C23: footprint Capacitor_SMD:C_0402_1005Metric -> Capacitor_SMD:C_0603_1608Metric
- C24, C8: value 100nF -> 0.1uF
- D1: value 22V -> BZX84C22-7-F
- D3, D4: value D_Schottky -> 1N4148
- J4: value Conn_01x02 -> 78171-0002
- J7: value OUTPUT -> 78171-0002
- Q1: value SSM3J340R -> SSM3J340R
- R10, R11, R12, R3, R4, R6, R9: footprint Resistor_SMD:R_0402_1005Metric -> Resistor_SMD:R_0603_1608Metric
- R2: footprint Resistor_SMD:R_0805_2012Metric -> Resistor_SMD:R_0603_1608Metric
- SW3: value SW_Push -> BTN_R
- U2: value W25Q32JVSS -> W25Q16JVUXIQ; footprint Finn-Lib:W25Q16FWUXIE -> Finn-Lib: USON-8_2x3x0.6mm
- moved C21 3.05 mm to (161.4, 75.8)
- moved C3 2.92 mm to (163.4, 75.8), turned to -90 degrees
- moved R6 0.54 mm to (144.4, 77.1)
- moved R11 0.51 mm to (149.0, 65.5)
- moved C23 0.46 mm to (141.0, 71.6)
- moved R10 0.46 mm to (146.6, 89.4)
- moved R3 0.40 mm to (144.8, 91.6)
- moved R8 0.38 mm to (142.9, 88.4)
- moved R4 0.28 mm to (161.8, 89.2)
- moved TP4 0.24 mm to (165.0, 88.5)
- moved U1 0.11 mm to (133.5, 77.1)
Connections:
- net /Reset renamed /User_RST
- C21 pad 2: Net-(U3-VI) -> Net-(D3-K)
- U3 pad 1: Net-(U3-VI) -> Net-(D3-K)
Routing:
- net Net-(D3-K): track 4.76 -> 11.6 mm
- net Net-(U3-VI): track 6.14 -> 0.00 mm
- net /FLASH_CS: track 15.0 -> 15.8 mm
- net /BOOT: track 3.21 -> 3.88 mm
- net /RUN: track 34.0 -> 33.5 mm
- net /CC1: track 39.0 -> 38.4 mm
- net +3.3V: track 41.2 -> 41.5 mm, vias 13 -> 12
- net GND: vias 150 -> 147
Other:
- board text removed: "3V3"

Commit message: docs
Parts:
- D1, R17, R18, R20, R21: moved to F.Cu
- SW3: value BTN_R -> BTN_UR
- moved R18 13.3 mm to (140.7, 72.5), turned to -90 degrees
- moved D1 11.9 mm to (138.2, 71.2), turned to -90 degrees
- moved R17 6.73 mm to (138.3, 74.0), turned to 0 degrees
- moved C23 1.55 mm to (142.2, 72.5), turned to 90 degrees
- moved TP8 1.28 mm to (132.8, 66.3)
Routing:
- net /V_{S}: track 16.6 -> 24.2 mm, vias 1 -> 2
- net VBUS: track 23.8 -> 18.3 mm
- net /CC2: track 33.6 -> 35.2 mm
- net /CC1: track 38.4 -> 39.8 mm
- net Net-(D1-A): track 1.88 -> 2.79 mm
- net /SCL_0: track 25.8 -> 25.4 mm, vias 2 -> 4
- net /SDA_0: track 26.0 -> 26.3 mm, vias 2 -> 4
- net GND: vias 147 -> 140
