File: PCB/Machine-Controller.kicad_sch (KiCad schematic)
At the start: 85 parts, among them J1 RESET, J2 Conn_01x05, J3 Conn_01x03, J4 Conn_01x02, J5 Conn_01x03, J6 USB_C_Receptacle_USB2.0, J7 OUTPUT, Q1 SSM3J340R, SW1 SW_SPDT, SW2 SW_Push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

Commit message: BoM and Docs
Parts:
- removed FBr1: FerriteBead, Capacitor_SMD:C_0805_2012Metric, symbol Device:FerriteBead_Small
- removed J1: RESET, Personalised:SW_SPST_TL3342, symbol Connector_Generic:Conn_01x02
- added SW4: BTN_R, Finn-Lib:SW_SPST_TL3342, symbol Switch:SW_Push
- C23: footprint Capacitor_SMD:C_0402_1005Metric -> Capacitor_SMD:C_0603_1608Metric
- C24, C8: value 100nF -> 0.1uF
- D1: value 22V -> BZX84C22-7-F
- D3, D4: value D_Schottky -> 1N4148
- D6: Alternative (none) -> PUSB3F96X
- J2: now not fitted; now left out of the parts list
- J4: value Conn_01x02 -> 78171-0002
- J7: value OUTPUT -> 78171-0002
- Q1: value SSM3J340R -> SSM3J340R; Alternative (none) -> IRLML5203TRPBF
- R10, R11, R12, R3, R4, R6, R9: footprint Resistor_SMD:R_0402_1005Metric -> Resistor_SMD:R_0603_1608Metric
- R2: footprint Resistor_SMD:R_0805_2012Metric -> Resistor_SMD:R_0603_1608Metric
- SW3: value SW_Push -> BTN_R
- TH1: now not fitted
- U1: Alternative (none) -> MT3608
- U2: value W25Q32JVSS -> W25Q16JVUXIQ; footprint Finn-Lib:W25Q16FWUXIE -> Finn-Lib: USON-8_2x3x0.6mm; Alternative (none) -> W25Q16xxx in USON-8 2x3mm
- U4: Alternative (none) -> N/A
Connections:
- net GND: now also SW4.1
- net RUN: now also SW4.2
- net at C3.2, D3.1 (K): now also C21.2, U3.1 (VI)
- net Reset renamed User_RST
Other:
- note added: "Load Disconnect using P-Channel MOSFET"
- note added: "No NMOS switch, Needs to work with non PD chargers"
- note added: "USB & TVS"
- note added: "USB-PD CONTROLLER"
- note removed: "+5V POWER"
- note removed: "Load Disconnect using P-Channel MOSFET (Q1)"
- note removed: "No NMOS switch, RP2040 needs power immediately Must work with non PD chargers"
- moved on the sheet: C10, C11, C12, C13, C14, C15, C18, C19, C22, C23, C24, C25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

Commit message: docs
Parts:
- SW3: value BTN_R -> BTN_UR
Changed lines of the file:
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@@
 			)
 		)
-		(property "Value" "BTN_R"
+		(property "Value" "BTN_UR"
 			(at 267.97 133.858 0)
 			(effects
